File: ThumbsUp.kicad_pcb (KiCad board)
At the start: 2 copper layers, 251.1 x 336.1 mm, 126 parts, among them J1 Conn_01x04_Male, J10 Raiser_Male, J11 Raiser_Female, J12 Raiser_Male, J13 Raiser_Female, J14 Raiser_Male, J15 Raiser_Female, J16 Raiser_Male, J17 Raiser_Female, J18 Raiser_Male, J19 52559-1233, J2 Conn_01x04_Male, J20 Conn_01x04_Female, J21 Conn_01x04_Female, J22 Conn_01x04_Female, J23 Conn_01x04_Female, J24 Conn_01x04_Male, J25 Conn_01x04_Male, J26 Conn_01x04_Male, J27 Conn_01x04_Male, J28 Conn_01x04_Female, J29 Conn_01x04_Female, J3 Conn_01x04_Female, J30 Conn_01x04_Female, J31 Conn_01x04_Female, J32 Battery, J4 Conn_01x04_Male, J5 Conn_01x04_Female, J6 Conn_01x04_Male, J7 Conn_01x04_Male, J8 Conn_01x04_Male, J9 Raiser_Female, SW1 SW_Push, SW2 SW_DIP_x01, U1 ProMicro

Commit message: Layed out switches and cross-plate connectors
Parts:
- removed G***: LOGO, Silkscreens:Crowfeet75
- removed J1, J2, J24, J25, J26, J27, J4, J6, J7, J8: Conn_01x04_Male, Connector_PinHeader_2.54mm:PinHeader_1x04_P2.54mm_Vertical
- removed J10, J12, J14, J16, J18: Raiser_Male, Connector_PinHeader_2.54mm:PinHeader_1x04_P2.54mm_Vertical
- removed J11, J13, J15, J17, J9: Raiser_Female, Connector_PinSocket_2.54mm:PinSocket_1x04_P2.54mm_Vertical
- removed J20, J21, J22, J23, J28, J29, J3, J30, J31, J5: Conn_01x04_Female, Connector_PinSocket_2.54mm:PinSocket_1x04_P2.54mm_Vertical
- added D45: D_Small, Diode_SMD:D_SOD-123, B.Cu at (94.3, 27.4)
- added D46: D_Small, Diode_SMD:D_SOD-123, B.Cu at (100.0, 27.4)
- added D47: D_Small, Diode_SMD:D_SOD-123, B.Cu at (105.8, 27.4)
- added D48: D_Small, Diode_SMD:D_SOD-123, B.Cu at (111.5, 27.4)
- added D49: D_Small, Diode_SMD:D_SOD-123, B.Cu at (117.3, 27.4)
- added D50: D_Small, Diode_SMD:D_SOD-123, B.Cu at (174.8, 27.4)
- added D51: D_Small, Diode_SMD:D_SOD-123, B.Cu at (123.0, 27.4)
- added D52: D_Small, Diode_SMD:D_SOD-123, B.Cu at (134.6, 27.4)
- added D53: D_Small, Diode_SMD:D_SOD-123, B.Cu at (140.3, 27.4)
- added D54: D_Small, Diode_SMD:D_SOD-123, B.Cu at (146.1, 27.4)
- added D55: D_Small, Diode_SMD:D_SOD-123, B.Cu at (151.8, 27.4)
- added D56: D_Small, Diode_SMD:D_SOD-123, B.Cu at (157.6, 27.4)
- added D57: D_Small, Diode_SMD:D_SOD-123, B.Cu at (163.3, 27.4)
- added D58: D_Small, Diode_SMD:D_SOD-123, B.Cu at (169.1, 27.4)
- added JF11: Raiser_Female, Connector_PinSocket_2.54mm:PinSocket_1x04_P2.54mm_Vertical, F.Cu at (49.0, 227.5)
- added JF13: Raiser_Female, Connector_PinSocket_2.54mm:PinSocket_1x04_P2.54mm_Vertical, F.Cu at (68.5, 63.0)
- added JF15: Raiser_Female, Connector_PinSocket_2.54mm:PinSocket_1x04_P2.54mm_Vertical, F.Cu at (75.5, 63.5)
- added JF17: Raiser_Female, Connector_PinSocket_2.54mm:PinSocket_1x04_P2.54mm_Vertical, F.Cu at (161.5, 231.5)
- added JF20: Conn_01x04_Female, Connector_PinSocket_2.54mm:PinSocket_1x04_P2.54mm_Vertical, F.Cu at (96.0, 164.5)
- added JF21: Conn_01x04_Female, Connector_PinSocket_2.54mm:PinSocket_1x04_P2.54mm_Vertical, F.Cu at (96.0, 183.5)
- added JF22: Conn_01x04_Female, Connector_PinSocket_2.54mm:PinSocket_1x04_P2.54mm_Vertical, F.Cu at (96.0, 202.5)
- added JF23: Conn_01x04_Female, Connector_PinSocket_2.54mm:PinSocket_1x04_P2.54mm_Vertical, F.Cu at (109.0, 239.0)
- added JF28: Conn_01x04_Female, Connector_PinSocket_2.54mm:PinSocket_1x04_P2.54mm_Vertical, F.Cu at (189.0, 202.5)
- added JF29: Conn_01x04_Female, Connector_PinSocket_2.54mm:PinSocket_1x04_P2.54mm_Vertical, F.Cu at (189.0, 183.5)
- added JF3: Conn_01x04_Female, Connector_PinSocket_2.54mm:PinSocket_1x04_P2.54mm_Vertical, F.Cu at (96.0, 145.5)
- added JF30: Conn_01x04_Female, Connector_PinSocket_2.54mm:PinSocket_1x04_P2.54mm_Vertical, F.Cu at (189.0, 164.5)
- added JF31: Conn_01x04_Female, Connector_PinSocket_2.54mm:PinSocket_1x04_P2.54mm_Vertical, F.Cu at (189.0, 145.5)
- added JF33: Conn_01x04_Female, Connector_PinSocket_2.54mm:PinSocket_1x04_P2.54mm_Vertical, F.Cu at (168.4, 239.0)
- added JF43: Conn_01x04_Female, Connector_PinSocket_2.54mm:PinSocket_1x04_P2.54mm_Vertical, F.Cu at (94.9, 239.0)
- added JF45: Conn_01x04_Female, Connector_PinSocket_2.54mm:PinSocket_1x04_P2.54mm_Vertical, F.Cu at (123.5, 231.5)
- added JF5: Conn_01x04_Female, Connector_PinSocket_2.54mm:PinSocket_1x04_P2.54mm_Vertical, F.Cu at (197.8, 239.0)
- added JF9: Raiser_Female, Connector_PinSocket_2.54mm:PinSocket_1x04_P2.54mm_Vertical, F.Cu at (236.0, 227.5)
- added JM11: Raiser_Male, Connector_PinHeader_2.54mm:PinHeader_1x04_P2.54mm_Vertical, B.Cu at (49.0, 227.5)
- added JM13: Raiser_Male, Connector_PinHeader_2.54mm:PinHeader_1x04_P2.54mm_Vertical, B.Cu at (68.5, 63.0)
- added JM15: Raiser_Male, Connector_PinHeader_2.54mm:PinHeader_1x04_P2.54mm_Vertical, B.Cu at (75.5, 63.5)
- added JM17: Raiser_Male, Connector_PinHeader_2.54mm:PinHeader_1x04_P2.54mm_Vertical, B.Cu at (161.5, 231.5)
- added JM20: Conn_01x04_Male, Connector_PinHeader_2.54mm:PinHeader_1x04_P2.54mm_Vertical, B.Cu at (96.0, 164.5)
- added JM21: Conn_01x04_Male, Connector_PinHeader_2.54mm:PinHeader_1x04_P2.54mm_Vertical, B.Cu at (96.0, 183.5)
- added JM22: Conn_01x04_Male, Connector_PinHeader_2.54mm:PinHeader_1x04_P2.54mm_Vertical, B.Cu at (96.0, 202.5)
- added JM23: Conn_01x04_Male, Connector_PinHeader_2.54mm:PinHeader_1x04_P2.54mm_Vertical, B.Cu at (109.0, 239.0)
- added JM28: Conn_01x04_Male, Connector_PinHeader_2.54mm:PinHeader_1x04_P2.54mm_Vertical, B.Cu at (189.0, 202.5)
- added JM29: Conn_01x04_Male, Connector_PinHeader_2.54mm:PinHeader_1x04_P2.54mm_Vertical, B.Cu at (189.0, 183.5)
- added JM3: Conn_01x04_Male, Connector_PinHeader_2.54mm:PinHeader_1x04_P2.54mm_Vertical, B.Cu at (96.0, 145.5)
- added JM30: Conn_01x04_Male, Connector_PinHeader_2.54mm:PinHeader_1x04_P2.54mm_Vertical, B.Cu at (189.0, 164.5)
- added JM31: Conn_01x04_Male, Connector_PinHeader_2.54mm:PinHeader_1x04_P2.54mm_Vertical, B.Cu at (189.0, 145.5)
- added JM33: Conn_01x04_Male, Connector_PinHeader_2.54mm:PinHeader_1x04_P2.54mm_Vertical, B.Cu at (168.4, 239.0)
- added JM43: Conn_01x04_Male, Connector_PinHeader_2.54mm:PinHeader_1x04_P2.54mm_Vertical, B.Cu at (94.9, 239.0)
- added JM45: Conn_01x04_Male, Connector_PinHeader_2.54mm:PinHeader_1x04_P2.54mm_Vertical, B.Cu at (123.5, 231.5)
- added JM5: Male, Connector_PinHeader_2.54mm:PinHeader_1x04_P2.54mm_Vertical, B.Cu at (197.8, 239.0)
- added JM9: Raiser_Male, Connector_PinHeader_2.54mm:PinHeader_1x04_P2.54mm_Vertical, B.Cu at (236.0, 227.5)
- added MX45: SwGrave, MX_Alps_Hybrid:MX-1U-NoLED_HotSwap, F.Cu at (19.0, 152.0)
- added MX46: Sw1, MX_Alps_Hybrid:MX-1U-NoLED_HotSwap, F.Cu at (38.0, 156.0)
- added MX47: Sw2, MX_Alps_Hybrid:MX-1U-NoLED_HotSwap, F.Cu at (57.0, 151.0)
- added MX48: Sw3, MX_Alps_Hybrid:MX-1U-NoLED_HotSwap, F.Cu at (76.0, 146.0)
- added MX49: Sw4, MX_Alps_Hybrid:MX-1U-NoLED_HotSwap, F.Cu at (95.0, 155.0)
- added MX50: Sw5, MX_Alps_Hybrid:MX-1U-NoLED_HotSwap, F.Cu at (114.0, 151.0)
- added MX51: SwThL, MX_Alps_Hybrid:MX-1U-NoLED_HotSwap, F.Cu at (133.0, 231.0)
- added MX52: Sw6, MX_Alps_Hybrid:MX-1U-NoLED_HotSwap, F.Cu at (171.0, 151.0)
- added MX53: SwThR, MX_Alps_Hybrid:MX-1U-NoLED_HotSwap, F.Cu at (152.0, 231.0)
- added MX54: Sw7, MX_Alps_Hybrid:MX-1U-NoLED_HotSwap, F.Cu at (190.0, 155.0)
- added MX55: Sw8, MX_Alps_Hybrid:MX-1U-NoLED_HotSwap, F.Cu at (209.0, 146.0)
- added MX56: Sw9, MX_Alps_Hybrid:MX-1U-NoLED_HotSwap, F.Cu at (228.0, 151.0)
- added MX57: Sw0, MX_Alps_Hybrid:MX-1U-NoLED_HotSwap, F.Cu at (247.0, 156.0)
- added MX58: SwDEL, MX_Alps_Hybrid:MX-1U-NoLED_HotSwap, F.Cu at (266.0, 152.0)
- MX1, MX10, MX11, MX12, MX13, MX14, MX15, MX16, MX17, MX18, MX19, MX2, MX20, MX21, MX22, MX23, MX24, MX25, MX26, MX27, MX28, MX29, MX3, MX30, MX31, MX32, MX33, MX34, MX35, MX36, MX37, MX38, MX39, MX4, MX40, MX41, MX42, MX43, MX44, MX5, MX6, MX7, MX8, MX9: footprint keyswitches:Kailh_socket_PG1350_optional -> MX_Alps_Hybrid:MX-1U-NoLED_HotSwap
- SW2: moved to B.Cu
- moved SW1 221.4 mm to (33.0, 46.0), turned to 180 degrees
- moved D40 216.5 mm to (65.5, 27.4), turned to 180 degrees
- moved D18 215.5 mm to (282.6, 95.0), turned to 180 degrees
- moved D19 214.4 mm to (276.9, 91.6), turned to 180 degrees
- moved U1 211.3 mm to (35.2, 6.74), turned to 0 degrees
- moved D43 211.1 mm to (82.8, 27.4), turned to 180 degrees
- moved D13 210.8 mm to (287.3, 103.8), turned to 180 degrees
- moved D44 209.3 mm to (88.5, 27.4), turned to 180 degrees
- moved D42 207.9 mm to (77.0, 27.4), turned to 180 degrees
- moved D14 206.7 mm to (262.4, 78.1), turned to 180 degrees
- moved D34 205.2 mm to (59.8, 27.4), turned to 180 degrees
- moved D32 204.8 mm to (71.3, 27.4), turned to 180 degrees
- moved D9 199.7 mm to (267.6, 87.0), turned to 180 degrees
- moved J32 195.1 mm to (267.0, 50.0), turned to 180 degrees
- moved D31 193.1 mm to (180.6, 27.6), turned to 180 degrees
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Connections:
- D1 pad 1: ROW0 -> ROWL1
- D10 pad 1: ROW2 -> ROWL3
- D11 pad 1: ROW2 -> ROWL3
- D12 pad 1: ROW2 -> ROWL3
- D13 pad 1: ROW3 -> ROWL4
- D14 pad 1: ROW3 -> ROWL4
- D15 pad 1: ROW0 -> ROWL1
- D16 pad 1: ROW1 -> ROWL2
- D17 pad 1: ROW2 -> ROWL3
- D18 pad 1: ROW3 -> ROWL4
- D19 pad 1: ROW3 -> ROWL4
- D2 pad 1: ROW0 -> ROWL1
- D20 pad 1: ROW0 -> ROWL1
- D21 pad 1: ROW1 -> ROWL2
- D22 pad 1: ROW2 -> ROWL3
- D23 pad 1: ROW0 -> ROWR1
- D24 pad 1: ROW1 -> ROWR2
- D25 pad 1: ROW2 -> ROWL0
- D26 pad 1: ROW0 -> ROWR1
- D27 pad 1: ROW1 -> ROWR2
- D28 pad 1: ROW2 -> ROWL0
- D29 pad 1: ROW3 -> ROWL0
- D3 pad 1: ROW0 -> ROWL1
- D30 pad 1: ROW3 -> ROWL0
- D31 pad 1: ROW0 -> ROWR1
- D32 pad 1: ROW0 -> ROWR1
- D33 pad 1: ROW0 -> ROWR1
- D34 pad 1: ROW0 -> ROWR1
- D35 pad 1: ROW1 -> ROWR2
- D36 pad 1: ROW1 -> ROWR2
- D37 pad 1: ROW1 -> ROWR2
- D38 pad 1: ROW1 -> ROWR2
- D39 pad 1: ROW2 -> ROWL0
- D4 pad 1: ROW0 -> ROWL1
- D40 pad 1: ROW2 -> ROWL0
- D41 pad 1: ROW2 -> ROWL0
- D42 pad 1: ROW2 -> ROWL0
- D43 pad 1: ROW3 -> ROWL0
- D44 pad 1: ROW3 -> ROWL0
- D5 pad 1: ROW1 -> ROWL2
- D6 pad 1: ROW1 -> ROWL2
- D7 pad 1: ROW1 -> ROWL2
- D8 pad 1: ROW1 -> ROWL2
- D9 pad 1: ROW2 -> ROWL3
- J19 pad 1: Net-(J19-Pad1) -> (no net)
- J19 pad 2: Net-(J19-Pad2) -> (no net)
- J19 pad 3: Net-(J19-Pad3) -> (no net)
- J19 pad 4: Net-(J19-Pad4) -> (no net)
- J19 pad 5: Net-(J19-Pad5) -> (no net)
- J19 pad 6: Net-(J19-Pad6) -> (no net)
- J19 pad 7: Net-(J19-Pad7) -> (no net)
- J19 pad 8: Net-(J19-Pad8) -> (no net)
- J19 pad MP1: Net-(J19-PadMP1) -> (no net)
- J19 pad MP2: Net-(J19-PadMP2) -> (no net)
- J19 pad MP3: Net-(J19-PadMP3) -> (no net)
- J19 pad MP4: Net-(J19-PadMP4) -> (no net)
- MX23 pad 1: COL6 -> COL5
- MX24 pad 1: COL6 -> COL5
- MX25 pad 1: COL6 -> COL5
- MX27 pad 1: COL7 -> COL4
- MX28 pad 1: COL7 -> COL4
- MX29 pad 1: COL7 -> COL4
- MX34 pad 1: COL8 -> COL3
- MX38 pad 1: COL9 -> COL2
- U1 pad 1: ROW0 -> COL0
- U1 pad 10: COL4 -> ROWL0
- U1 pad 11: COL3 -> ROWL1
- U1 pad 12: COL2 -> ROWL2
- U1 pad 13: COL1 -> (no net)
- U1 pad 14: COL0 -> (no net)
- U1 pad 15: COL6 -> (no net)
- U1 pad 16: COLB -> ROWR2
- U1 pad 17: COLA -> ROWR1
- U1 pad 18: COL9 -> ROWR0
- U1 pad 19: COL8 -> ROWL4
- U1 pad 2: ROW1 -> COL1
- U1 pad 20: COL7 -> ROWL3
- U1 pad 3: Net-(U1-Pad3) -> GND
- U1 pad 4: Net-(U1-Pad4) -> GND
- U1 pad 7: ROW2 -> COL2
- U1 pad 8: ROW3 -> COL3
Routing:
- net COL6: track 172.0 -> 0.00 mm, vias 3 -> 0
- net COL8: track 155.4 -> 0.00 mm, vias 1 -> 0
- net COL7: track 152.6 -> 0.00 mm, vias 2 -> 0
- net ROW3: track 150.6 -> 0.00 mm, vias 2 -> 0
- net COL4: track 149.6 -> 0.00 mm, vias 1 -> 0
- net GND: track 148.5 -> 0.00 mm
- net COL5: track 140.2 -> 0.00 mm, vias 2 -> 0
- net ROW2: track 136.3 -> 0.00 mm, vias 2 -> 0
- net COL9: track 135.9 -> 0.00 mm, vias 1 -> 0
- net Net-(JF20-Pad4): track 130.2 -> 0.00 mm, vias 1 -> 0
- net COL3: track 127.2 -> 0.00 mm, vias 1 -> 0
- net Net-(JF28-Pad4): track 126.8 -> 0.00 mm
- net COL0: track 123.9 -> 0.00 mm, vias 1 -> 0
- net COL1: track 121.8 -> 0.00 mm, vias 1 -> 0
- net COLA: track 117.1 -> 0.00 mm, vias 1 -> 0
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Other:
- board outline removed
- board text removed: "Battery +RED HERE"
- board text removed: "Place ProMicro face to the plate."
- board text removed: "QMK: #define MATRIX_ROW_PINS {D3, D2, D4, C6} #define MATRIX_COL_PINS {B2, B6, B5, B4, E6, D7, B3, F4, F5, F6, F7, B1} #define DIODE_DIRECTION COL2ROW"
- board text removed: "RESET"
- board text removed: "Thumbs Up! by Sasha Karmanov October 28, 2022 https://github.com/ak66666/ ThumbsUpUnsplitV2ProMicro"
- board text removed: "|<"

Commit message: Rotated the wings into 44 degree position, added the external boundary
Parts:
- moved D1 319.9 mm to (158.8, 345.9)
- moved D12 319.9 mm to (84.0, 345.9)
- moved D22 319.9 mm to (216.3, 346.1)
- moved D31 319.9 mm to (210.6, 346.1)
- moved D32 319.9 mm to (101.3, 345.9)
- moved D34 319.9 mm to (89.8, 345.9)
- moved D40 319.9 mm to (95.5, 345.9)
- moved D42 319.9 mm to (107.0, 345.9)
- moved D43 319.9 mm to (112.8, 345.9)
- moved D44 319.9 mm to (118.5, 345.9)
- moved D45 319.9 mm to (124.3, 345.9)
- moved D46 319.9 mm to (130.1, 345.9)
- moved D47 319.9 mm to (135.8, 345.9)
- moved D48 319.9 mm to (141.6, 345.9)
- moved D49 319.9 mm to (147.3, 345.9)
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Connections:
- JF11 pad 1: GND -> (no net)
- JF11 pad 4: (no net) -> GND
- JM11 pad 1: GND -> (no net)
Other:
- board outline added: 280.6 x 148.8 mm

Commit message: Arranged the cross-board headers and sockets
Parts:
- moved JM13 361.0 mm to (142.5, -171.5)
- moved JM17 361.0 mm to (189.1, -106.0)
- moved JM43 361.0 mm to (71.6, -115.0)
- moved JM45 361.0 mm to (95.9, -106.0)
- moved JM5 361.0 mm to (219.5, -119.5)
- moved MX18 361.0 mm to (88.7, -112.2)
- moved MX22 361.0 mm to (73.5, -123.6)
- moved MX26 361.0 mm to (211.5, -123.6)
- moved MX30 361.0 mm to (196.4, -112.1)
- moved MX51 361.0 mm to (103.8, -100.7)
- moved MX53 361.0 mm to (181.2, -100.7)
- moved JF13 190.0 mm to (142.5, -0.50)
- moved JF17 190.0 mm to (189.1, 65.0)
- moved JF43 190.0 mm to (71.6, 56.0)
- moved JF45 190.0 mm to (95.9, 65.0)
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Other:
- board size 280.6 x 148.8 mm -> 280.6 x 468.6 mm

Commit message: Routed L1 PCB
Parts:
- moved R2 383.4 mm to (520.6, 48.1)
- moved D1 383.4 mm to (415.8, 61.4)
- moved D10 383.4 mm to (445.8, 29.8)
- moved D11 383.4 mm to (491.7, 52.5)
- moved D12 383.4 mm to (341.1, 61.4)
- moved D13 383.4 mm to (530.3, 53.9)
- moved D14 383.4 mm to (505.4, 28.1)
- moved D15 383.4 mm to (525.6, 48.3)
- moved D16 383.4 mm to (491.7, 55.8)
- moved D17 383.4 mm to (471.3, 13.2)
- moved D18 383.4 mm to (525.6, 45.0)
- moved D19 383.4 mm to (519.9, 41.6)
- moved D2 383.4 mm to (505.4, 21.4)
- moved D20 383.4 mm to (485.9, 52.5)
- moved D21 383.4 mm to (496.1, 15.1)
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Connections:
- D39 pad 2: Net-(D39-Pad2) -> (no net)
- D40 pad 2: Net-(D40-Pad2) -> (no net)
- D41 pad 2: Net-(D41-Pad2) -> (no net)
- D42 pad 2: Net-(D42-Pad2) -> (no net)
- JF11 pad 2: GND -> L1GND
- JF11 pad 3: GND -> L1GND
- JF11 pad 4: GND -> L1GND
- JF15 pad 1: GND -> L1GND
- JF15 pad 2: GND -> L1GND
- JF15 pad 3: GND -> L1GND
- JF15 pad 4: GND -> L1GND
- JF9 pad 1: GND -> L1GND
- JF9 pad 2: GND -> L1GND
- JF9 pad 3: GND -> L1GND
- JF9 pad 4: GND -> L1GND
- JM13 pad 1: GND -> L3GND
- JM13 pad 2: GND -> L3GND
- JM13 pad 3: GND -> L3GND
- JM13 pad 4: GND -> L3GND
- JM20 pad 1: COL3 -> COL0
- JM20 pad 2: COL2 -> COL1
- JM20 pad 3: COL1 -> COL2
- JM20 pad 4: COL0 -> COL3
- JM21 pad 1: Net-(D4-Pad2) -> Net-(D1-Pad2)
- JM21 pad 2: Net-(D3-Pad2) -> Net-(D2-Pad2)
- JM21 pad 3: Net-(D2-Pad2) -> Net-(D3-Pad2)
- JM21 pad 4: Net-(D1-Pad2) -> Net-(D4-Pad2)
- JM22 pad 1: Net-(D8-Pad2) -> Net-(D5-Pad2)
- JM22 pad 2: Net-(D7-Pad2) -> Net-(D6-Pad2)
- JM22 pad 3: Net-(D6-Pad2) -> Net-(D7-Pad2)
- JM22 pad 4: Net-(D5-Pad2) -> Net-(D8-Pad2)
- JM28 pad 1: COL3 -> (no net)
- JM28 pad 2: COL2 -> (no net)
- JM28 pad 3: COL1 -> (no net)
- JM28 pad 4: COL0 -> (no net)
- JM29 pad 1: Net-(D34-Pad2) -> Net-(D38-Pad2)
- JM29 pad 2: Net-(D33-Pad2) -> Net-(D37-Pad2)
- JM29 pad 3: Net-(D32-Pad2) -> Net-(D36-Pad2)
- JM29 pad 4: Net-(D31-Pad2) -> Net-(D35-Pad2)
- JM3 pad 1: Net-(D45-Pad2) -> Net-(D48-Pad2)
- JM3 pad 2: Net-(D46-Pad2) -> Net-(D47-Pad2)
- JM3 pad 3: Net-(D47-Pad2) -> Net-(D46-Pad2)
- JM3 pad 4: Net-(D48-Pad2) -> Net-(D45-Pad2)
- JM30 pad 1: Net-(D38-Pad2) -> Net-(D34-Pad2)
- JM30 pad 2: Net-(D37-Pad2) -> Net-(D33-Pad2)
- JM30 pad 3: Net-(D36-Pad2) -> Net-(D32-Pad2)
- JM30 pad 4: Net-(D35-Pad2) -> Net-(D31-Pad2)
- JM31 pad 1: Net-(D42-Pad2) -> Net-(D58-Pad2)
- JM31 pad 2: Net-(D41-Pad2) -> Net-(D57-Pad2)
- JM31 pad 3: Net-(D40-Pad2) -> Net-(D56-Pad2)
- JM31 pad 4: Net-(D39-Pad2) -> Net-(D55-Pad2)
- JM33 pad 1: Net-(D58-Pad2) -> COL3
- JM33 pad 2: Net-(D57-Pad2) -> COL2
- JM33 pad 3: Net-(D56-Pad2) -> COL1
- JM33 pad 4: Net-(D55-Pad2) -> COL0
- MX1 pad 1: Net-(JF20-Pad4) -> Net-(JF20-Pad1)
- MX1 pad 2: Net-(JF21-Pad1) -> Net-(JF21-Pad4)
- MX11 pad 1: Net-(JF20-Pad1) -> Net-(JF20-Pad4)
- MX11 pad 2: Net-(JF21-Pad4) -> Net-(JF21-Pad1)
- MX12 pad 1: Net-(JF20-Pad1) -> Net-(JF20-Pad4)
- MX12 pad 2: Net-(JF22-Pad4) -> Net-(JF22-Pad1)
- MX13 pad 1: Net-(JF20-Pad1) -> Net-(JF20-Pad4)
- MX2 pad 1: Net-(JF20-Pad4) -> Net-(JF20-Pad1)
- MX2 pad 2: Net-(JF22-Pad1) -> Net-(JF22-Pad4)
- MX3 pad 1: Net-(JF20-Pad4) -> Net-(JF20-Pad1)
- MX31 pad 1: Net-(JF28-Pad1) -> Net-(JF33-Pad1)
- MX31 pad 2: Net-(JF29-Pad4) -> Net-(JF30-Pad4)
- MX32 pad 1: Net-(JF28-Pad1) -> Net-(JF33-Pad1)
- MX32 pad 2: Net-(JF30-Pad4) -> Net-(JF29-Pad4)
- MX33 pad 1: Net-(JF28-Pad1) -> Net-(JF33-Pad1)
- MX33 pad 2: Net-(JF31-Pad4) -> Net-(JF28-Pad4)
- MX35 pad 1: Net-(JF28-Pad2) -> Net-(JF33-Pad2)
- MX35 pad 2: Net-(JF29-Pad3) -> Net-(JF30-Pad3)
- MX36 pad 1: Net-(JF28-Pad2) -> Net-(JF33-Pad2)
- MX36 pad 2: Net-(JF30-Pad3) -> Net-(JF29-Pad3)
- MX37 pad 1: Net-(JF28-Pad2) -> Net-(JF33-Pad2)
- MX37 pad 2: Net-(JF31-Pad3) -> Net-(JF28-Pad3)
- MX39 pad 1: Net-(JF28-Pad3) -> Net-(JF33-Pad3)
- MX39 pad 2: Net-(JF29-Pad2) -> Net-(JF30-Pad2)
- MX4 pad 1: Net-(JF20-Pad3) -> Net-(JF20-Pad2)
- MX4 pad 2: Net-(JF21-Pad2) -> Net-(JF21-Pad3)
- MX40 pad 1: Net-(JF28-Pad3) -> Net-(JF33-Pad3)
- MX40 pad 2: Net-(JF30-Pad2) -> Net-(JF29-Pad2)
- MX41 pad 1: Net-(JF28-Pad3) -> Net-(JF33-Pad3)
- MX41 pad 2: Net-(JF31-Pad2) -> Net-(JF28-Pad2)
- MX42 pad 1: Net-(JF28-Pad4) -> Net-(JF33-Pad4)
- MX42 pad 2: Net-(JF29-Pad1) -> Net-(JF30-Pad1)
- MX43 pad 1: Net-(JF28-Pad4) -> Net-(JF33-Pad4)
- MX43 pad 2: Net-(JF30-Pad1) -> Net-(JF29-Pad1)
- MX44 pad 1: Net-(JF28-Pad4) -> Net-(JF33-Pad4)
- MX44 pad 2: Net-(JF31-Pad1) -> Net-(JF28-Pad1)
- MX45 pad 1: Net-(JF20-Pad4) -> Net-(JF20-Pad1)
- MX45 pad 2: Net-(JF3-Pad4) -> Net-(JF3-Pad1)
- MX46 pad 1: Net-(JF20-Pad3) -> Net-(JF20-Pad2)
- MX46 pad 2: Net-(JF3-Pad3) -> Net-(JF3-Pad2)
- MX47 pad 1: Net-(JF20-Pad2) -> Net-(JF20-Pad3)
- MX47 pad 2: Net-(JF3-Pad2) -> Net-(JF3-Pad3)
- MX48 pad 1: Net-(JF20-Pad1) -> Net-(JF20-Pad4)
- MX48 pad 2: Net-(JF3-Pad1) -> Net-(JF3-Pad4)
- MX5 pad 1: Net-(JF20-Pad3) -> Net-(JF20-Pad2)
- MX5 pad 2: Net-(JF22-Pad2) -> Net-(JF22-Pad3)
- MX55 pad 1: Net-(JF28-Pad1) -> Net-(JF33-Pad1)
- MX55 pad 2: Net-(JF33-Pad4) -> Net-(JF31-Pad4)
- MX56 pad 1: Net-(JF28-Pad2) -> Net-(JF33-Pad2)
- MX56 pad 2: Net-(JF33-Pad3) -> Net-(JF31-Pad3)
- MX57 pad 1: Net-(JF28-Pad3) -> Net-(JF33-Pad3)
- MX57 pad 2: Net-(JF33-Pad2) -> Net-(JF31-Pad2)
- MX58 pad 1: Net-(JF28-Pad4) -> Net-(JF33-Pad4)
- MX58 pad 2: Net-(JF33-Pad1) -> Net-(JF31-Pad1)
- MX6 pad 1: Net-(JF20-Pad3) -> Net-(JF20-Pad2)
- MX7 pad 1: Net-(JF20-Pad2) -> Net-(JF20-Pad3)
- MX7 pad 2: Net-(JF21-Pad3) -> Net-(JF21-Pad2)
- MX8 pad 1: Net-(JF20-Pad2) -> Net-(JF20-Pad3)
- MX8 pad 2: Net-(JF22-Pad3) -> Net-(JF22-Pad2)
- MX9 pad 1: Net-(JF20-Pad2) -> Net-(JF20-Pad3)
Routing:
- net Net-(JF33-Pad4): track 0.00 -> 177.8 mm
- net Net-(JF20-Pad1): track 0.00 -> 163.7 mm
- net Net-(JF33-Pad3): track 0.00 -> 156.0 mm
- net Net-(JF33-Pad2): track 0.00 -> 145.7 mm
- net Net-(JF20-Pad2): track 0.00 -> 140.2 mm
- net Net-(JF33-Pad1): track 0.00 -> 139.0 mm
- net Net-(JF20-Pad3): track 0.00 -> 117.4 mm
- net Net-(JF31-Pad1): track 0.00 -> 110.2 mm
- net Net-(JF23-Pad1): track 0.00 -> 108.7 mm
- net Net-(JF3-Pad1): track 0.00 -> 103.4 mm
- net Net-(JF29-Pad1): track 0.00 -> 98.2 mm
- net Net-(JF30-Pad1): track 0.00 -> 97.6 mm
- net Net-(JF28-Pad1): track 0.00 -> 97.0 mm
- net Net-(JF31-Pad2): track 0.00 -> 95.9 mm
- net Net-(JF22-Pad4): track 0.00 -> 95.2 mm
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- added copper zone on B.Cu, net L1GND
Other:
- board text added: "Put ProMicro Face to PCB."

Commit message: Routed L2 PCB
Parts:
- removed JF15: Raiser_Female, Connector_PinSocket_2.54mm:PinSocket_1x04_P2.54mm_Vertical
- removed JM15: Raiser_Male, Connector_PinHeader_2.54mm:PinHeader_1x04_P2.54mm_Vertical
- removed SW1: SW_Push, random-keyboard-parts:SKQG-1155865
- added S1: BUTT-4, BUTT-4:BUTT4, F.Cu at (172.7, 75.0)
- moved D18 452.8 mm to (72.8, 45.4), turned to 90 degrees
- moved D13 450.2 mm to (80.2, 45.4), turned to 90 degrees
- moved D19 444.6 mm to (75.3, 45.4), turned to 90 degrees
- moved D14 428.1 mm to (77.7, 45.4), turned to 90 degrees
- moved D7 424.3 mm to (95.6, 45.4), turned to 90 degrees
- moved D9 418.1 mm to (92.9, 54.3), turned to 270 degrees
- moved D5 409.8 mm to (90.4, 45.4), turned to 90 degrees
- moved D6 407.4 mm to (93.0, 45.4), turned to 90 degrees
- moved D11 403.7 mm to (88.0, 54.3), turned to 270 degrees
- moved D2 402.8 mm to (103.3, 45.4), turned to 90 degrees
- moved D15 402.4 mm to (123.4, 38.1)
- moved D3 399.1 mm to (106.0, 45.4), turned to 90 degrees
- moved D8 393.7 mm to (98.2, 45.4), turned to 90 degrees
- moved D17 390.0 mm to (82.6, 45.4), turned to 90 degrees
- moved D22 388.6 mm to (85.1, 45.4), turned to 90 degrees
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Connections:
- D25 pad 1: ROWL0 -> ROWR3
- D28 pad 1: ROWL0 -> ROWR3
- D29 pad 1: ROWL0 -> ROWR4
- D30 pad 1: ROWL0 -> ROWR4
- D39 pad 1: ROWL0 -> ROWR3
- D39 pad 2: (no net) -> Net-(D39-Pad2)
- D40 pad 1: ROWL0 -> ROWR3
- D40 pad 2: (no net) -> Net-(D40-Pad2)
- D41 pad 1: ROWL0 -> ROWR3
- D41 pad 2: (no net) -> Net-(D41-Pad2)
- D42 pad 1: ROWL0 -> ROWR3
- D42 pad 2: (no net) -> Net-(D42-Pad2)
- D43 pad 1: ROWL0 -> ROWR4
- D44 pad 1: ROWL0 -> ROWR4
- D53 pad 1: ROWL0 -> ROWR4
- JM11 pad 1: (no net) -> Net-(D14-Pad2)
- JM28 pad 1: (no net) -> Net-(D42-Pad2)
- JM28 pad 2: (no net) -> Net-(D41-Pad2)
- JM28 pad 3: (no net) -> Net-(D40-Pad2)
- JM28 pad 4: (no net) -> Net-(D39-Pad2)
- U1 pad 1: COL0 -> COL3
- U1 pad 10: ROWL0 -> ROWL1
- U1 pad 11: ROWL1 -> ROWL0
- U1 pad 13: (no net) -> COL4
- U1 pad 14: (no net) -> ROWR4
- U1 pad 15: (no net) -> ROWR3
- U1 pad 2: COL1 -> COL2
- U1 pad 7: COL2 -> COL1
- U1 pad 8: COL3 -> COL0
Routing:
- net GND: track 0.00 -> 410.9 mm, vias 0 -> 1
- net COL4: track 0.00 -> 400.1 mm, vias 0 -> 5
- net COL2: track 0.00 -> 364.5 mm, vias 0 -> 5
- net COL3: track 0.00 -> 360.1 mm, vias 0 -> 9
- net COL5: track 0.00 -> 327.4 mm, vias 0 -> 4
- net COL1: track 0.00 -> 184.4 mm, vias 0 -> 2
- net COL0: track 0.00 -> 178.6 mm, vias 0 -> 2
- net ROWR4: track 0.00 -> 145.3 mm
- net SDA: track 0.00 -> 131.5 mm, vias 0 -> 1
- net ROWL4: track 0.00 -> 126.5 mm, vias 0 -> 1
- net SCL: track 0.00 -> 120.9 mm, vias 0 -> 1
- net ROWL3: track 0.00 -> 116.9 mm, vias 0 -> 1
- net Net-(JM45-Pad1): track 0.00 -> 113.7 mm
- net VCC: track 0.00 -> 112.1 mm
- net Net-(JM45-Pad2): track 0.00 -> 108.3 mm
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Other:
- outline, holes or cut-outs redrawn
- board text added: "-->|--"
- board text added: "ThumbsUp! v5 MX ProMicro u/ak66666 May 22, 2023"

Commit message: Added mounting holes, enlarged ProMicro pin holes to fit machined sockets.
Parts:
- added H1: MountingHole_Pad, MountingHole:MountingHole_6mm_Pad_Via, F.Cu at (142.4, 215.2)
- added H2: MountingHole_Pad, MountingHole:MountingHole_8.4mm_M8_Pad_Via, F.Cu at (142.4, 234.6)

Commit message: Fixed the thumbcluster connections.
Connections:
- JF43 pad 1: COL3 -> COL4
- JF43 pad 4: COL4 -> COL5
- JF45 pad 1: COL5 -> COL1
- JF45 pad 4: COL5 -> COL1
- JF5 pad 1: COL4 -> COL5
- JF5 pad 4: COL3 -> COL4
Routing:
- net COL5: track 327.4 -> 406.0 mm, vias 4 -> 6
- net COL1: track 184.4 -> 232.3 mm
- net COL3: track 360.1 -> 337.2 mm, vias 9 -> 8
- net COL4: track 400.1 -> 386.8 mm
- net GND: track 410.9 -> 405.7 mm
- net COL2: track 364.5 -> 359.7 mm
